Commit message: Add a physical-feasibility gate for fitted link mass parameters
calibration/feasibility.py checks gravity-tier parameters [m, m*c] per link:
positive mass, centre of mass inside a box from the URDF collision geometry
(or a padded kinematic hull when the meshes cannot be loaded), total mass
within 0.8x-2.5x the URDF, and a gripper allowance on the end link.

Without data, audit() only checks pointwise. Given the fit's regressor and
torques, it separates a nullspace artifact (a feasible set fits as well)
from real infeasibility, and reports the regressor rank and per-parameter
nullspace fractions behind that call. project() runs two convex stages:
best feasible fit, then the point nearest the URDF within 5% of that
residual. It is never called implicitly.

The module imports neither pinocchio nor scipy at load time; LinkSpec and
ParamSet are plain data with a mandatory units="SI". PiperModel.link_specs()
and gravity_regressor() build the inputs in-package. TauExtEstimator warns
on unphysical inertial_overrides, piper-diagnose --urdf audits them, and
the identification summary states the feasibility result. The full tier
(pseudo-inertia LMI) is an interface only; docs/feasibility.md explains why
static data cannot use it.

File: tests/fixtures/toy6.urdf (robot description, URDF)
Before this commit: robot toy6, 7 links, 6 joints
Links:
- link link2: geometry collision box size=0.06 0.06 0.32
- link link3: geometry collision cylinder length=0.27 radius=0.03
